File: attenuator/attenuator_block.kicad_sch (KiCad schematic)
At the start: 11 parts, among them U11 4259-63, U12 4259-63

Commit message: pcb improve it
Parts:
- C19: renamed from C23; footprint Capacitor_SMD:C_0805_2012Metric -> Capacitor_SMD:C_0603_1608Metric
- C20: renamed from C24; footprint Capacitor_SMD:C_0805_2012Metric -> Capacitor_SMD:C_0603_1608Metric
- C21: renamed from C25; footprint Capacitor_SMD:C_0805_2012Metric -> Capacitor_SMD:C_0603_1608Metric
- C22: renamed from C26; footprint Capacitor_SMD:C_0805_2012Metric -> Capacitor_SMD:C_0603_1608Metric
- R10: renamed from R12; footprint Resistor_SMD:R_0805_2012Metric_Pad1.20x1.40mm_HandSolder -> Resistor_SMD:R_0603_1608Metric_Pad0.98x0.95mm_HandSolder
- R1_A4: renamed from R1_A5; footprint Resistor_SMD:R_0805_2012Metric_Pad1.20x1.40mm_HandSolder -> Resistor_SMD:R_0603_1608Metric_Pad0.98x0.95mm_HandSolder
- R2_A4: renamed from R2_A5; footprint Resistor_SMD:R_0805_2012Metric_Pad1.20x1.40mm_HandSolder -> Resistor_SMD:R_0603_1608Metric_Pad0.98x0.95mm_HandSolder
- R9: renamed from R11; footprint Resistor_SMD:R_0805_2012Metric_Pad1.20x1.40mm_HandSolder -> Resistor_SMD:R_0603_1608Metric_Pad0.98x0.95mm_HandSolder
- Rs_A4: renamed from Rs_A5; footprint Resistor_SMD:R_0805_2012Metric_Pad1.20x1.40mm_HandSolder -> Resistor_SMD:R_0603_1608Metric_Pad0.98x0.95mm_HandSolder
- renumbered U12 to U10, U11 to U9

Commit message: finish simulation and kicad
Parts:
- added C26: GCQ1555C1HR85WB01D, attenuator:CAPC1005X55N, symbol c_switch:GCQ1555C1HR85WB01D
- added L1: LQG15HN2N0S02D, attenuator:INDC1005X55N, symbol l_switch:LQG15HN2N0S02D
Connections:
- net GND: now also C26.1
- net RFC_IN: now also C26.2, L1.1; no longer C19.1, U9.5 (RFC)
- new net: C19.1, L1.2, U9.5 (RFC)
Other:
- moved on the sheet: C19, C20
Changed lines of the file:
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@@
   (junction (at 133.35 69.85) (diameter 0) (color 0 0 0 0)
   )
-  (junction (at 36.83 67.31) (diameter 0) (color 0 0 0 0)
+  (junction (at 41.91 67.31) (diameter 0) (color 0 0 0 0)
+  )
+  (junction (at 25.4 67.31) (diameter 0) (color 0 0 0 0)
   )
   (junction (at 214.63 67.31) (diameter 0) (color 0 0 0 0)
@@
     (stroke (width 0) (type default))
   )
-  (wire (pts (xy 31.75 67.31) (xy 36.83 67.31))
-    (stroke (width 0) (type default))
-  )
-  (wire (pts (xy 36.83 67.31) (xy 46.99 67.31))
-    (stroke (width 0) (type default))
-  )
-  (wire (pts (xy 36.83 74.93) (xy 36.83 67.31))
+  (wire (pts (xy 24.13 67.31) (xy 25.4 67.31))
+    (stroke (width 0) (type default))
+  )
+  (wire (pts (xy 41.91 74.93) (xy 41.91 67.31))
     (stroke (width 0) (type default))
   )
@@
     (stroke (width 0) (type default))
   )
-  (wire (pts (xy 36.83 92.71) (xy 36.83 95.25))
+  (wire (pts (xy 41.91 92.71) (xy 41.91 95.25))
     (stroke (width 0) (type default))
   )
@@
     (stroke (width 0) (type default))
   )
+  (wire (pts (xy 25.4 78.74) (xy 25.4 85.09))
+    (stroke (width 0) (type default))
+  )
   (wire (pts (xy 133.35 81.28) (xy 133.35 83.82))
     (stroke (width 0) (type default))
@@
     (stroke (width 0) (type default))
   )
-  (wire (pts (xy 36.83 82.55) (xy 36.83 85.09))
+  (wire (pts (xy 41.91 82.55) (xy 41.91 85.09))
+    (stroke (width 0) (type default))
+  )
+  (wire (pts (xy 41.91 67.31) (xy 46.99 67.31))
+    (stroke (width 0) (type default))
+  )
+  (wire (pts (xy 25.4 67.31) (xy 26.67 67.31))
+    (stroke (width 0) (type default))
+  )
+  (wire (pts (xy 40.64 67.31) (xy 41.91 67.31))
     (stroke (width 0) (type default))
   )
   (wire (pts (xy 115.57 69.85) (xy 115.57 73.66))
+    (stroke (width 0) (type default))
+  )
+  (wire (pts (xy 25.4 67.31) (xy 25.4 71.12))
     (stroke (width 0) (type default))
   )
@@
     (effects (font (size 1.27 1.27)) (justify left))
   )
-  (hierarchical_label "RFC_IN" (shape input) (at 31.75 67.31 180) (fields_autoplaced)
+  (hierarchical_label "RFC_IN" (shape input) (at 24.13 67.31 180) (fields_autoplaced)
     (effects (font (size 1.27 1.27)) (justify right))
   )
@@
         (path "/3b0f5433-415e-45c9-9c4a-85a692e565e5/3da84243-0db9-493d-afe7-bbdf34a70e6f"
           (reference "#PWR021") (unit 1)
+        )
+      )
+    )
+  )
+  (symbol (lib_id "c_switch:GCQ1555C1HR85WB01D") (at 25.4 76.2 90) (unit 1)
+    (in_bom yes) (on_board yes) (dnp no)
+    (property "Reference" "C26" (at 29.21 73.66 90)
+      (effects (font (size 1.27 1.27)) (justify right))
+    )
+    (property "Value" "GCQ1555C1HR85WB01D" (at 29.21 76.2 90)
+      (effects (font (size 1.27 1.27)) (justify right))
+    )
+    (property "Footprint" "attenuator:CAPC1005X55N" (at 25.4 76.2 0)
+      (effects (font (size 1.27 1.27)) (justify bottom) hide)
+    )
+    (property "Datasheet" "" (at 25.4 76.2 0)
+      (effects (font (size 1.27 1.27)) hide)
+    )
+    (pin "1")
+    (pin "2")
+    (instances
+      (project "attenuator"
+        (path "/3b0f5433-415e-45c9-9c4a-85a692e565e5/d8a81011-8742-4aef-8bd1-0388c515e538"
+          (reference "C26") (unit 1)
+        )
+        (path "/3b0f5433-415e-45c9-9c4a-85a692e565e5/b0edad66-e740-4e6d-bc3a-542edbe7ee2e"
+          (reference "C23") (unit 1)
+        )
+        (path "/3b0f5433-415e-45c9-9c4a-85a692e565e5/c52d33fc-f0f4-4621-a7b6-5f1c2bd6a0f4"
+          (reference "C24") (unit 1)
+        )
+        (path "/3b0f5433-415e-45c9-9c4a-85a692e565e5/3da84243-0db9-493d-afe7-bbdf34a70e6f"
+          (reference "C25") (unit 1)
         )
       )
@@
     )
   )
+  (symbol (lib_id "l_switch:LQG15HN2N0S02D") (at 34.29 67.31 0) (unit 1)
+    (in_bom yes) (on_board yes) (dnp no) (fields_autoplaced)
+    (property "Reference" "L1" (at 34.29 60.96 0)
+      (effects (font (size 1.27 1.27)))
+    )
+    (property "Value" "LQG15HN2N0S02D" (at 34.29 63.5 0)
+      (effects (font (size 1.27 1.27)))
+    )
+    (property "Footprint" "attenuator:INDC1005X55N" (at 34.29 67.31 0)
+      (effects (font (size 1.27 1.27)) (justify bottom) hide)
+    )
+    (property "Datasheet" "" (at 34.29 67.31 0)
+      (effects (font (size 1.27 1.27)) hide)
+    )
+    (pin "1")
+    (pin "2")
+    (instances
+      (project "attenuator"
+        (path "/3b0f5433-415e-45c9-9c4a-85a692e565e5/b0edad66-e740-4e6d-bc3a-542edbe7ee2e"
+          (reference "L1") (unit 1)
+        )
+        (path "/3b0f5433-415e-45c9-9c4a-85a692e565e5/c52d33fc-f0f4-4621-a7b6-5f1c2bd6a0f4"
+          (reference "L2") (unit 1)
+        )
+        (path "/3b0f5433-415e-45c9-9c4a-85a692e565e5/3da84243-0db9-493d-afe7-bbdf34a70e6f"
+          (reference "L3") (unit 1)
+        )
+        (path "/3b0f5433-415e-45c9-9c4a-85a692e565e5/d8a81011-8742-4aef-8bd1-0388c515e538"
+          (reference "L4") (unit 1)
+        )
+      )
+    )
+  )
   (symbol (lib_id "Device:R") (at 115.57 77.47 0) (unit 1)
     (in_bom yes) (on_board yes) (dnp no) (fields_autoplaced)
@@
     )
   )
-  (symbol (lib_id "power:GND") (at 36.83 95.25 0) (unit 1)
-    (in_bom yes) (on_board yes) (dnp no) (fields_autoplaced)
-    (property "Reference" "#PWR029" (at 36.83 101.6 0)
-      (effects (font (size 1.27 1.27)) hide)
-    )
-    (property "Value" "GND" (at 36.83 100.33 0)
-      (effects (font (size 1.27 1.27)))
-    )
-    (property "Footprint" "" (at 36.83 95.25 0)
-      (effects (font (size 1.27 1.27)) hide)
-    )
-    (property "Datasheet" "" (at 36.83 95.25 0)
+  (symbol (lib_id "power:GND") (at 41.91 95.25 0) (unit 1)
+    (in_bom yes) (on_board yes) (dnp no) (fields_autoplaced)
+    (property "Reference" "#PWR029" (at 41.91 101.6 0)
+      (effects (font (size 1.27 1.27)) hide)
+    )
+    (property "Value" "GND" (at 41.91 100.33 0)
+      (effects (font (size 1.27 1.27)))
+    )
+    (property "Footprint" "" (at 41.91 95.25 0)
+      (effects (font (size 1.27 1.27)) hide)
+    )
+    (property "Datasheet" "" (at 41.91 95.25 0)
       (effects (font (size 1.27 1.27)) hide)
     )
@@
     )
   )
-  (symbol (lib_id "Device:C") (at 36.83 88.9 0) (unit 1)
+  (symbol (lib_id "Device:C") (at 41.91 88.9 0) (unit 1)
     (in_bom yes) (on_board yes) (dnp no)
-    (property "Reference" "C20" (at 30.48 88.9 0)
-      (effects (font (size 1.27 1.27)) (justify left))
-    )
-    (property "Value" "0.5p" (at 30.48 91.44 0)
-      (effects (font (size 1.27 1.27)) (justify left))
-    )
-    (property "Footprint" "Capacitor_SMD:C_0603_1608Metric" (at 37.7952 92.71 0)
-      (effects (font (size 1.27 1.27)) hide)
-    )
-    (property "Datasheet" "~" (at 36.83 88.9 0)
+    (property "Reference" "C20" (at 35.56 88.9 0)
+      (effects (font (size 1.27 1.27)) (justify left))
+    )
+    (property "Value" "0.5p" (at 35.56 91.44 0)
+      (effects (font (size 1.27 1.27)) (justify left))
+    )
+    (property "Footprint" "Capacitor_SMD:C_0603_1608Metric" (at 42.8752 92.71 0)
+      (effects (font (size 1.27 1.27)) hide)
+    )
+    (property "Datasheet" "~" (at 41.91 88.9 0)
       (effects (font (size 1.27 1.27)) hide)
     )
@@
     )
   )
-  (symbol (lib_id "Device:C") (at 36.83 78.74 0) (unit 1)
+  (symbol (lib_id "power:GND") (at 25.4 85.09 0) (unit 1)
+    (in_bom yes) (on_board yes) (dnp no) (fields_autoplaced)
+    (property "Reference" "#PWR039" (at 25.4 91.44 0)
+      (effects (font (size 1.27 1.27)) hide)
+    )
+    (property "Value" "GND" (at 25.4 90.17 0)
+      (effects (font (size 1.27 1.27)))
+    )
+    (property "Footprint" "" (at 25.4 85.09 0)
+      (effects (font (size 1.27 1.27)) hide)
+    )
+    (property "Datasheet" "" (at 25.4 85.09 0)
+      (effects (font (size 1.27 1.27)) hide)
+    )
+    (pin "1")
+    (instances
+      (project "attenuator"
+        (path "/3b0f5433-415e-45c9-9c4a-85a692e565e5/b0edad66-e740-4e6d-bc3a-542edbe7ee2e"
+          (reference "#PWR039") (unit 1)
+        )
+        (path "/3b0f5433-415e-45c9-9c4a-85a692e565e5/c52d33fc-f0f4-4621-a7b6-5f1c2bd6a0f4"
+          (reference "#PWR040") (unit 1)
+        )
+        (path "/3b0f5433-415e-45c9-9c4a-85a692e565e5/3da84243-0db9-493d-afe7-bbdf34a70e6f"
+          (reference "#PWR041") (unit 1)
+        )
+        (path "/3b0f5433-415e-45c9-9c4a-85a692e565e5/d8a81011-8742-4aef-8bd1-0388c515e538"
+          (reference "#PWR042") (unit 1)
+        )
+      )
+    )
+  )
+  (symbol (lib_id "Device:C") (at 41.91 78.74 0) (unit 1)
     (in_bom yes) (on_board yes) (dnp no)
-    (property "Reference" "C19" (at 30.48 78.74 0)
-      (effects (font (size 1.27 1.27)) (justify left))
-    )
-    (property "Value" "0.5p" (at 30.48 81.28 0)
-      (effects (font (size 1.27 1.27)) (justify left))
-    )
-    (property "Footprint" "Capacitor_SMD:C_0603_1608Metric" (at 37.7952 82.55 0)
-      (effects (font (size 1.27 1.27)) hide)
-    )
-    (property "Datasheet" "~" (at 36.83 78.74 0)
-      (effects (font (size 1.27 1.27)) hide)
-    )
+    (property "Reference" "C19" (at 35.56 78.74 0)
+      (effects (font (size 1.27 1.27)) (justify left))
+    )
+    (property "Value" "0.5p" (at 35.56 81.28 0)
+      (effects (font (size 1.27 1.27)) (justify left))
+    )
+    (property "Footprint" "Capacitor_SMD:C_0603_1608Metric" (at 42.8752 82.55 0)
+      (effects (font (size 1.27 1.27)) hide)
+    )
+    (property "Datasheet" "~" (at 41.91 78.74 0)
+      (effects (font (size 1.27 1.27)) hide)
+    )
