File: attenuator/attenuator_block_v2.kicad_sch (KiCad schematic)
At the start: 12 parts, among them U10 4259-63, U9 4259-63

Commit message: pcb improve it
Parts:
- C15: renamed from C19; footprint Capacitor_SMD:C_0805_2012Metric -> Capacitor_SMD:C_0603_1608Metric
- C16: renamed from C20; footprint Capacitor_SMD:C_0805_2012Metric -> Capacitor_SMD:C_0603_1608Metric
- C17: renamed from C21; footprint Capacitor_SMD:C_0805_2012Metric -> Capacitor_SMD:C_0603_1608Metric
- C18: renamed from C22; footprint Capacitor_SMD:C_0805_2012Metric -> Capacitor_SMD:C_0603_1608Metric
- R1_E1, R2_E1, Rs_E1, Rs_E2: footprint Resistor_SMD:R_0805_2012Metric_Pad1.20x1.40mm_HandSolder -> Resistor_SMD:R_0603_1608Metric_Pad0.98x0.95mm_HandSolder
- R7: renamed from R9; footprint Resistor_SMD:R_0805_2012Metric_Pad1.20x1.40mm_HandSolder -> Resistor_SMD:R_0603_1608Metric_Pad0.98x0.95mm_HandSolder
- R8: renamed from R10; footprint Resistor_SMD:R_0805_2012Metric_Pad1.20x1.40mm_HandSolder -> Resistor_SMD:R_0603_1608Metric_Pad0.98x0.95mm_HandSolder
- renumbered U9 to U7, U10 to U8

Commit message: finish simulation and kicad
Parts:
- added C27: GCQ1555C1HR85WB01D, attenuator:CAPC1005X55N, symbol c_switch:GCQ1555C1HR85WB01D
- added L6: LQG15HN2N0S02D, attenuator:INDC1005X55N, symbol l_switch:LQG15HN2N0S02D
Connections:
- net GND: now also C27.1
- net RFC_IN: now also C27.2, L6.1; no longer C15.1, U7.5 (RFC)
- new net: C15.1, L6.2, U7.5 (RFC)
Changed lines of the file:
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@@
 (kicad_sch (version 20230121) (generator eeschema)
   (paper "A4")
+  (junction (at 38.1 76.2) (diameter 0) (color 0 0 0 0)
+  )
   (junction (at 57.15 76.2) (diameter 0) (color 0 0 0 0)
   )
@@
     (stroke (width 0) (type default))
   )
-  (wire (pts (xy 52.07 76.2) (xy 57.15 76.2))
+  (wire (pts (xy 34.29 76.2) (xy 38.1 76.2))
     (stroke (width 0) (type default))
   )
@@
     (stroke (width 0) (type default))
   )
+  (wire (pts (xy 53.34 76.2) (xy 57.15 76.2))
+    (stroke (width 0) (type default))
+  )
   (wire (pts (xy 137.16 82.55) (xy 143.51 82.55))
     (stroke (width 0) (type default))
@@
     (stroke (width 0) (type default))
   )
+  (wire (pts (xy 38.1 87.63) (xy 38.1 93.98))
+    (stroke (width 0) (type default))
+  )
   (wire (pts (xy 157.48 82.55) (xy 157.48 78.74))
     (stroke (width 0) (type default))
@@
   )
   (wire (pts (xy 137.16 82.55) (xy 137.16 85.09))
+    (stroke (width 0) (type default))
+  )
+  (wire (pts (xy 38.1 80.01) (xy 38.1 76.2))
     (stroke (width 0) (type default))
   )
@@
     (effects (font (size 1.27 1.27)) (justify left))
   )
-  (hierarchical_label "RFC_IN" (shape input) (at 52.07 76.2 180) (fields_autoplaced)
+  (hierarchical_label "RFC_IN" (shape input) (at 34.29 76.2 180) (fields_autoplaced)
     (effects (font (size 1.27 1.27)) (justify right))
   )
@@
     )
   )
+  (symbol (lib_id "l_switch:LQG15HN2N0S02D") (at 45.72 76.2 0) (unit 1)
+    (in_bom yes) (on_board yes) (dnp no) (fields_autoplaced)
+    (property "Reference" "L6" (at 45.72 69.85 0)
+      (effects (font (size 1.27 1.27)))
+    )
+    (property "Value" "LQG15HN2N0S02D" (at 45.72 72.39 0)
+      (effects (font (size 1.27 1.27)))
+    )
+    (property "Footprint" "attenuator:INDC1005X55N" (at 45.72 76.2 0)
+      (effects (font (size 1.27 1.27)) (justify bottom) hide)
+    )
+    (property "Datasheet" "" (at 45.72 76.2 0)
+      (effects (font (size 1.27 1.27)) hide)
+    )
+    (pin "1")
+    (pin "2")
+    (instances
+      (project "attenuator"
+        (path "/3b0f5433-415e-45c9-9c4a-85a692e565e5/1814b441-73d1-4a6f-9de4-def20b8dedaa"
+          (reference "L6") (unit 1)
+        )
+      )
+    )
+  )
   (symbol (lib_id "rf_switch:4259-63") (at 118.11 78.74 180) (unit 1)
     (in_bom yes) (on_board yes) (dnp no) (fields_autoplaced)
@@
     )
   )
+  (symbol (lib_id "power:GND") (at 38.1 93.98 0) (unit 1)
+    (in_bom yes) (on_board yes) (dnp no) (fields_autoplaced)
+    (property "Reference" "#PWR043" (at 38.1 100.33 0)
+      (effects (font (size 1.27 1.27)) hide)
+    )
+    (property "Value" "GND" (at 38.1 99.06 0)
+      (effects (font (size 1.27 1.27)))
+    )
+    (property "Footprint" "" (at 38.1 93.98 0)
+      (effects (font (size 1.27 1.27)) hide)
+    )
+    (property "Datasheet" "" (at 38.1 93.98 0)
+      (effects (font (size 1.27 1.27)) hide)
+    )
+    (pin "1")
+    (instances
+      (project "attenuator"
+        (path "/3b0f5433-415e-45c9-9c4a-85a692e565e5/1814b441-73d1-4a6f-9de4-def20b8dedaa"
+          (reference "#PWR043") (unit 1)
+        )
+      )
+    )
+  )
   (symbol (lib_id "power:GND") (at 57.15 104.14 0) (unit 1)
     (in_bom yes) (on_board yes) (dnp no) (fields_autoplaced)
@@
         )
       )
+    )
+  )
+  (symbol (lib_id "c_switch:GCQ1555C1HR85WB01D") (at 38.1 85.09 90) (unit 1)
+    (in_bom yes) (on_board yes) (dnp no)
+    (property "Reference" "C27" (at 41.91 82.55 90)
+      (effects (font (size 1.27 1.27)) (justify right))
+    )
+    (property "Value" "GCQ1555C1HR85WB01D" (at 41.91 85.09 90)
+      (effects (font (size 1.27 1.27)) (justify right))
+    )
+    (property "Footprint" "attenuator:CAPC1005X55N" (at 38.1 85.09 0)
+      (effects (font (size 1.27 1.27)) (justify bottom) hide)
+    )
+    (property "Datasheet" "" (at 38.1 85.09 0)
+      (effects (font (size 1.27 1.27)) hide)
+    )
+    (pin "1")
+    (pin "2")
+    (instances
+      (project "attenuator"
+        (path "/3b0f5433-415e-45c9-9c4a-85a692e565e5/1814b441-73d1-4a6f-9de4-def20b8dedaa"
+          (reference "C27") (unit 1)
+        )
+      )
